File: hardware/dumbwatch.kicad_sch (KiCad schematic)
At the start: 12 parts, among them J1 USB_C_Receptacle_USB2.0, J2 Programming Connector, U1 PIC18F27J53_ISS, Y1 32.768 kHz

Commit message: PCB rev 1 complete
Parts:
- removed J1: USB_C_Receptacle_USB2.0, Connector_USB:USB_C_Receptacle_GCT_USB4085, symbol Connector:USB_C_Receptacle_USB2.0
- removed R2, R3: 5.1k, Resistor_SMD:R_0805_2012Metric_Pad1.20x1.40mm_HandSolder, symbol Device:R_US
- added J1: USB_B_Micro, Connector_USB:USB_Micro-B_Amphenol_10104110_Horizontal, symbol Connector:USB_B_Micro
Connections:
- net +5V: now also J1.1 (VBUS)
- net BATT_SENS: now also U1.13 (RC2/AN11); no longer U1.4 (RA2/AN2)
- net BUSY: now also U1.26 (RB5/SDA1); no longer U1.2 (RA0/AN0)
- net CHRG_STAT: now also U1.3 (RA1/AN1); no longer U1.25 (RB4/SCL1)
- net D+: now also J1.3 (D+)
- net D-: now also J1.2 (D-)
- net GND: now also R1.1, J1.5 (GND); no longer R1.2
- net OSC1: now also U1.12 (RC1/T1OSI); no longer U1.11 (RC0/T1OSO)
- net OSC2: now also U1.11 (RC0/T1OSO); no longer U1.12 (RC1/T1OSI)
- net RESET: now also U1.25 (RB4/SCL1); no longer U1.3 (RA1/AN1)
- net USB_IN: now also U1.4 (RA2/AN2); no longer U1.26 (RB5/SDA1)
- new net: J1.6 (Shield), R1.2
- no-connect marks 9 -> 8
Other:
- moved on the sheet: R1
