File: hardware/eink.kicad_sch (KiCad schematic)
At the start: 20 parts, among them J3 EINK, Q1 DMG3418L-7

Commit message: PCB rev 1 complete
Parts:
- Q1: footprint Package_TO_SOT_SMD:SOT-23_Handsoldering -> Package_TO_SOT_SMD:SOT-23
Changed lines of the file:
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@@
       (effects (font (size 1.27 1.27)) (justify left))
     )
-    (property "Footprint" "Package_TO_SOT_SMD:SOT-23_Handsoldering" (id 2) (at 90.17 58.42 0)
+    (property "Footprint" "Package_TO_SOT_SMD:SOT-23" (id 2) (at 90.17 58.42 0)
       (effects (font (size 1.27 1.27)) hide)
     )
