File: hardware/power.kicad_sch (KiCad schematic)
At the start: 21 parts, among them J4 JST PH, Q2 NXV65UPR, U2 NCP115, U3 MCP73832T-2

Commit message: PCB rev 1 complete
Parts:
- Q2: footprint Package_TO_SOT_SMD:SOT-23_Handsoldering -> Package_TO_SOT_SMD:SOT-23
- U2: footprint Package_TO_SOT_SMD:TSOT-23-5_HandSoldering -> Package_TO_SOT_SMD:TSOT-23-5
- U3: footprint Package_TO_SOT_SMD:SOT-23-5_HandSoldering -> Package_TO_SOT_SMD:SOT-23-5
Changed lines of the file:
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@@
     (property "Reference" "U2" (id 0) (at 213.36 61.121 0))
     (property "Value" "NCP115" (id 1) (at 213.36 63.6579 0))
-    (property "Footprint" "Package_TO_SOT_SMD:TSOT-23-5_HandSoldering" (id 2) (at 213.36 68.58 0)
+    (property "Footprint" "Package_TO_SOT_SMD:TSOT-23-5" (id 2) (at 213.36 68.58 0)
       (effects (font (size 1.27 1.27)) hide)
     )
@@
       (effects (font (size 1.27 1.27)) (justify left))
     )
-    (property "Footprint" "Package_TO_SOT_SMD:SOT-23_Handsoldering" (id 2) (at 194.31 55.88 0)
+    (property "Footprint" "Package_TO_SOT_SMD:SOT-23" (id 2) (at 194.31 55.88 0)
       (effects (font (size 1.27 1.27)) hide)
     )
@@
     (property "Reference" "U3" (id 0) (at 217.17 120.811 0))
     (property "Value" "MCP73832T-2" (id 1) (at 217.17 123.3479 0))
-    (property "Footprint" "Package_TO_SOT_SMD:SOT-23-5_HandSoldering" (id 2) (at 217.17 130.81 0)
-      (effects (font (size 1.27 1.27)) hide)
-    )
+    (property "Footprint" "Package_TO_SOT_SMD:SOT-23-5" (id 2) (at 217.17 130.81 0)
+      (effects (font (size 1.27 1.27)) hide)
+    )
